File: BalthazarKeyboard.kicad_pcb (KiCad board)
At the start: 2 copper layers, 93 parts, among them J1 PSU I2C bus, SW1 ESC, SW10 2, SW2 F1, SW3 F2, SW39 SPACE, SW4 F3, SW5 F4, SW6 F5, SW7 F6, SW8 ¸¨, SW9 1!, U1 Pro Micro

Commit message: Add files via upload
Parts:
- removed D1, D10, D11, D12, D13, D14, D15, D16, D17, D18, D19, D2, D20, D21, D22, D23, D24, D25, D26, D27, D28, D29, D3, D30, D31, D32, D33, D34, D35, D36, D37, D38, D39, D4, D40, D41, D42, D43, D44, D45, D46, D47, D48, D49, D5, D50, D51, D52, D53, D54, D55, D56, D57, D58, D59, D6, D60, D61, D62, D63, D64, D65, D66, D67, D68, D69, D7, D70, D71, D72, D73, D74, D75, D76, D77, D8, D9: D, Diode_SMD:D_0805_2012Metric
- removed J1: PSU I2C bus, Connector_PinSocket_2.54mm:PinSocket_1x06_P2.54mm_Horizontal
- removed R8, R9: 200, Resistor_SMD:R_1206_3216Metric
- removed the SW39 at (128.3, 162.6)
- removed the SW39 at (193.0, 162.6)
- removed U1: Pro Micro, Module:Arduino_ProMicro
- added SW11: 3#, Button_Switch_THT:SW_PUSH_6mm_8mm, F.Cu at (95.0, 92.2)
- added SW12: 4$, Button_Switch_THT:SW_PUSH_6mm_8mm, F.Cu at (114.3, 94.0)
- added SW13: 5%, Button_Switch_THT:SW_PUSH_6mm_8mm, F.Cu at (133.6, 95.5)
- added SW14: 6&, Button_Switch_THT:SW_PUSH_6mm_8mm, F.Cu at (152.9, 97.3)
- added SW15: TAB, Button_Switch_Keyboard:SW_Cherry_MX_1.25u_Plate, F.Cu at (10.4, 75.2)
- added SW15: TAB, Button_Switch_THT:SW_PUSH_6mm_8mm, F.Cu at (17.8, 74.2)
- added SW16: Q, Button_Switch_Keyboard:SW_Cherry_MX_1.00u_Plate, F.Cu at (56.6, 99.6)
- added SW16: Q, Button_Switch_THT:SW_PUSH_6mm_8mm, F.Cu at (56.4, 101.3)
- added SW17: W, Button_Switch_THT:SW_PUSH_6mm_8mm, F.Cu at (75.7, 106.7)
- added SW18: E, Button_Switch_THT:SW_PUSH_6mm_8mm, F.Cu at (95.0, 111.5)
- added SW19: R, Button_Switch_THT:SW_PUSH_6mm_8mm, F.Cu at (114.3, 113.3)
- added SW20: T, Button_Switch_THT:SW_PUSH_6mm_8mm, F.Cu at (133.6, 115.6)
- added SW21: Y/Z, Button_Switch_THT:SW_PUSH_6mm_8mm, F.Cu at (152.9, 116.6)
- added SW22: CAPS, Button_Switch_THT:SW_PUSH_6mm_8mm, F.Cu at (17.8, 96.3)
- added SW23: A, Button_Switch_THT:SW_PUSH_6mm_8mm, F.Cu at (56.4, 120.7)
- added SW24: S, Button_Switch_THT:SW_PUSH_6mm_8mm, F.Cu at (75.7, 126.0)
- added SW25: D, Button_Switch_THT:SW_PUSH_6mm_8mm, F.Cu at (95.0, 130.8)
- added SW26: F, Button_Switch_THT:SW_PUSH_6mm_8mm, F.Cu at (114.3, 132.6)
- added SW27: G, Button_Switch_THT:SW_PUSH_6mm_8mm, F.Cu at (133.6, 134.9)
- added SW28: H, Button_Switch_THT:SW_PUSH_6mm_8mm, F.Cu at (152.9, 135.9)
- added SW29: SHIFT, Button_Switch_THT:SW_PUSH_6mm_8mm, F.Cu at (37.1, 98.6)
- added SW30: <>, Button_Switch_THT:SW_PUSH_6mm_8mm, F.Cu at (56.4, 140.0)
- added SW31: Y/Z, Button_Switch_THT:SW_PUSH_6mm_8mm, F.Cu at (75.7, 142.0)
- added SW32: X, Button_Switch_THT:SW_PUSH_6mm_8mm, F.Cu at (95.0, 150.1)
- added SW33: C, Button_Switch_THT:SW_PUSH_6mm_8mm, F.Cu at (114.3, 151.6)
- added SW34: V, Button_Switch_THT:SW_PUSH_6mm_8mm, F.Cu at (133.6, 153.4)
- added SW35: B, Button_Switch_THT:SW_PUSH_6mm_8mm, F.Cu at (152.9, 155.2)
- added SW36: CTRL, Button_Switch_Keyboard:SW_Cherry_MX_1.25u_PCB, F.Cu at (10.4, 118.9)
- added SW36: CTRL, Button_Switch_THT:SW_PUSH_6mm_8mm, F.Cu at (17.8, 117.6)
- added SW37: ALT, Button_Switch_THT:SW_PUSH_6mm_8mm, F.Cu at (37.1, 117.9)
- added SW38: Win/Apple, Button_Switch_Keyboard:SW_Cherry_MX_1.25u_PCB, F.Cu at (30.0, 148.3)
- added SW38: Win/Apple, Button_Switch_THT:SW_PUSH_6mm_8mm, F.Cu at (34.8, 139.7)
- added SW39: SPACE, Button_Switch_Keyboard:SW_Cherry_MX_2.00u_PCB, F.Cu at (47.2, 157.5)
- added SW40: LEFT, Button_Switch_THT:SW_PUSH_6mm_8mm, F.Cu at (249.4, 158.5)
- added SW41: DOWN, Button_Switch_THT:SW_PUSH_6mm_8mm, F.Cu at (268.7, 157.5)
- added SW42: RIGHT, Button_Switch_THT:SW_PUSH_6mm_8mm, F.Cu at (288.0, 158.8)
- added SW43: F7, Button_Switch_Keyboard:SW_Cherry_MX_1.00u_PCB, F.Cu at (167.6, 74.4)
- added SW43: F7, Button_Switch_THT:SW_PUSH_6mm_8mm, F.Cu at (167.4, 76.2)
- added SW44: F8, Button_Switch_Keyboard:SW_Cherry_MX_1.00u_PCB, F.Cu at (186.9, 69.6)
- added SW44: F8, Button_Switch_THT:SW_PUSH_6mm_8mm, F.Cu at (186.7, 71.1)
- added SW45: F9, Button_Switch_Keyboard:SW_Cherry_MX_1.00u_PCB, F.Cu at (206.2, 66.3)
- added SW45: F9, Button_Switch_THT:SW_PUSH_6mm_8mm, F.Cu at (206.0, 68.1)
- added SW46: F10, Button_Switch_Keyboard:SW_Cherry_MX_1.00u_PCB, F.Cu at (225.6, 62.7)
- added SW46: F10, Button_Switch_THT:SW_PUSH_6mm_8mm, F.Cu at (225.3, 64.5)
- added SW47: F11, Button_Switch_Keyboard:SW_Cherry_MX_1.00u_PCB, F.Cu at (244.9, 59.2)
- added SW47: F11, Button_Switch_THT:SW_PUSH_6mm_8mm, F.Cu at (244.6, 61.0)
- added SW48: F12, Button_Switch_Keyboard:SW_Cherry_MX_1.00u_PCB, F.Cu at (264.2, 55.9)
- added SW48: F12, Button_Switch_THT:SW_PUSH_6mm_8mm, F.Cu at (263.9, 57.7)
- added SW49: F13 PRTSCR, Button_Switch_Keyboard:SW_Cherry_MX_1.25u_PCB, F.Cu at (286.0, 50.8)
- added SW49: F13 PRTSCR, Button_Switch_THT:SW_PUSH_6mm_8mm, F.Cu at (285.8, 52.6)
- added SW50: 7/, Button_Switch_THT:SW_PUSH_6mm_8mm, F.Cu at (172.2, 95.5)
- added SW51: 8(, Button_Switch_THT:SW_PUSH_6mm_8mm, F.Cu at (191.5, 94.2)
- added SW52: 9), Button_Switch_THT:SW_PUSH_6mm_8mm, F.Cu at (210.8, 92.5)
- added SW53: 0=, Button_Switch_THT:SW_PUSH_6mm_8mm, F.Cu at (230.1, 86.4)
- added SW54: /?, Button_Switch_THT:SW_PUSH_6mm_8mm, F.Cu at (249.4, 81.3)
- added SW55: +*, Button_Switch_THT:SW_PUSH_6mm_8mm, F.Cu at (268.7, 80.3)
- added SW56: DELETE, Button_Switch_THT:SW_PUSH_6mm_8mm, F.Cu at (288.0, 71.9)
- added SW57: U, Button_Switch_THT:SW_PUSH_6mm_8mm, F.Cu at (172.2, 114.8)
- added SW58: I, Button_Switch_THT:SW_PUSH_6mm_8mm, F.Cu at (191.5, 113.5)
- added SW59: O, Button_Switch_THT:SW_PUSH_6mm_8mm, F.Cu at (210.8, 111.8)
- added SW60: P, Button_Switch_THT:SW_PUSH_6mm_8mm, F.Cu at (230.1, 105.7)
- added SW61: Š, Button_Switch_THT:SW_PUSH_6mm_8mm, F.Cu at (249.4, 100.6)
- added SW62: Đ, Button_Switch_THT:SW_PUSH_6mm_8mm, F.Cu at (268.7, 99.6)
- added SW63: BACKSPACE, Button_Switch_THT:SW_PUSH_6mm_8mm, F.Cu at (288.0, 91.2)
- added SW64: J, Button_Switch_THT:SW_PUSH_6mm_8mm, F.Cu at (172.2, 134.1)
- added SW65: K, Button_Switch_THT:SW_PUSH_6mm_8mm, F.Cu at (191.5, 132.8)
- added SW66: L, Button_Switch_THT:SW_PUSH_6mm_8mm, F.Cu at (210.8, 131.1)
- added SW67: Č, Button_Switch_THT:SW_PUSH_6mm_8mm, F.Cu at (230.1, 125.0)
- added SW68: Ć, Button_Switch_THT:SW_PUSH_6mm_8mm, F.Cu at (249.4, 119.9)
- added SW69: Ž, Button_Switch_THT:SW_PUSH_6mm_8mm, F.Cu at (268.7, 118.9)
- added SW70: ENTER, Button_Switch_THT:SW_PUSH_6mm_8mm, F.Cu at (288.0, 115.3)
- added SW71: N, Button_Switch_THT:SW_PUSH_6mm_8mm, F.Cu at (172.2, 153.4)
- added SW72: M, Button_Switch_THT:SW_PUSH_6mm_8mm, F.Cu at (191.5, 152.1)
- added SW73: ,;, Button_Switch_THT:SW_PUSH_6mm_8mm, F.Cu at (210.8, 150.4)
- added SW74: .:, Button_Switch_THT:SW_PUSH_6mm_8mm, F.Cu at (230.1, 144.3)
- added SW75: -_, Button_Switch_THT:SW_PUSH_6mm_8mm, F.Cu at (249.4, 139.2)
- added SW76: UP, Button_Switch_THT:SW_PUSH_6mm_8mm, F.Cu at (268.7, 138.2)
- added SW77: SHIFT, Button_Switch_THT:SW_PUSH_6mm_8mm, F.Cu at (288.0, 139.4)
- SW1: footprint Button_Switch_THT:SW_PUSH_6mm_8mm -> Button_Switch_Keyboard:SW_Cherry_MX_1.25u_PCB
- SW10, SW8, SW9: footprint Button_Switch_THT:SW_PUSH_6mm_8mm -> Button_Switch_Keyboard:SW_Cherry_MX_1.00u_Plate
- SW2, SW3, SW4, SW5, SW6, SW7: footprint Button_Switch_THT:SW_PUSH_6mm_8mm -> Button_Switch_Keyboard:SW_Cherry_MX_1.00u_PCB
- moved SW10 15.9 mm to (75.9, 85.6), turned to 0 degrees
- moved SW9 14.5 mm to (56.6, 80.3), turned to 0 degrees
- moved SW8 14.2 mm to (37.3, 77.5), turned to 0 degrees
- moved SW7 6.97 mm to (141.0, 82.0)
- moved SW1 6.35 mm to (20.3, 50.8), turned to 0 degrees
- moved SW4 2.33 mm to (80.5, 63.0), turned to 0 degrees
- moved SW3 2.10 mm to (61.2, 61.0), turned to 0 degrees
- moved SW5 1.48 mm to (99.8, 66.0), turned to 0 degrees
- moved SW6 1.02 mm to (119.1, 69.8), turned to 0 degrees
- moved SW2 1.02 mm to (41.9, 58.2), turned to 0 degrees
Routing:
- net (no net): track 0.00 -> 235.2 mm
- net row3: track 408.0 -> 191.9 mm
- net row2: track 377.3 -> 240.9 mm
- net Net-(D30-Pad2): track 14.6 -> 132.0 mm
- net row1: track 368.4 -> 257.3 mm
- net Net-(D38-Pad2): track 14.5 -> 125.6 mm
Other:
- board outline added: 289.6 x 127 mm
- board text added: "Balthazar"
- board text added: "______________________"
