File: BalthazarPSU.kicad_pcb (KiCad board)
At the start: 2 copper layers, 83.8 x 31.8 mm, 88 parts, among them IC1 BQ24193, J1 AudioIN, J10 3.3V/5V, J11 3.3V/5V, J3 thermistor, J4 AudioOUT, J5 USB_A_female, J6 USB_OTG_female, J7 host (promicro), J8 - VSYS1 +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

Commit message: Add files via upload
Parts:
- BATT1: renamed from - BATT +
- CBUS3a1, CBUS3a2, CBUS3a3, CPMID1a1: footprint Capacitor_SMD:C_0603_1608Metric -> Capacitor_SMD:C_0805_2012Metric
- FBEAD2, FBEAD3: footprint Inductor_SMD:L_Neosid_MicroCoil_Ms36-M -> Inductor_SMD:L_Neosid_MicroCoil_Ms36-L
- J8: value - VSYS1 + -> 3.3V 4A
- J9: renamed from - VSYS2 +
- PSU1: value - 9-12V + -> 3.9 - 17V adapter 3-5A
- renumbered J3 to THERM1
Connections:
- U2 pad 0: PGND -> Net-(U2-Pad0)
Routing:
- net PGND: track 482.6 -> 469.2 mm
- added copper zone on F.Cu, net Net-(FBEAD3-Pad2)
- removed copper zone on F.Cu, net Net-(BATT1-Pad1)
