File: BalthazarPSU.sch (KiCad schematic (older format))
At the start: 88 parts, among them IC1 BQ24193, J1 AudioIN, J10 3.3V/5V, J11 3.3V/5V, J4 AudioOUT, J5 USB_A_female, J6 USB_OTG_female, J7 host (promicro), J8 3.3V 4A, J9 3.3V 4A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

Commit message: Add files via upload
Parts:
- D1, D2, D4, D5: symbol BalthazarPSU-rescue:Led_Small -> BalthazarPSU-rescue:Led_Small-BalthazarPSU-rescue
- FBEAD2, FBEAD3, L1, L2, L3: symbol BalthazarPSU-rescue:INDUCTOR_SMALL -> BalthazarPSU-rescue:INDUCTOR_SMALL-BalthazarPSU-rescue
- IC1: symbol BalthazarPSU-rescue:BQ24193 -> BalthazarPSU-rescue:BQ24193-BalthazarPSU-rescue
- THERMISTOR(103-AT)1: symbol BalthazarPSU-rescue:THERMISTOR -> BalthazarPSU-rescue:THERMISTOR-BalthazarPSU-rescue
- renumbered BATT to BATT1, THERM to THERM1
Changed lines of the file:
@@
 $EndDescr
 $Comp
-L BalthazarPSU-rescue:INDUCTOR_SMALL L1
+L BalthazarPSU-rescue:INDUCTOR_SMALL-BalthazarPSU-rescue L1
 U 1 1 5E346E06
 P 5150 3300
@@
 $EndComp
 $Comp
-L BalthazarPSU-rescue:Led_Small D1
+L BalthazarPSU-rescue:Led_Small-BalthazarPSU-rescue D1
 U 1 1 5E347A22
 P 3550 3900
@@
 $EndComp
 $Comp
-L BalthazarPSU-rescue:Led_Small D2
+L BalthazarPSU-rescue:Led_Small-BalthazarPSU-rescue D2
 U 1 1 5E347A6B
 P 3550 4000
@@
 Connection ~ 4900 4900
 $Comp
-L BalthazarPSU-rescue:THERMISTOR THERMISTOR(103-AT)1
+L BalthazarPSU-rescue:THERMISTOR-BalthazarPSU-rescue THERMISTOR(103-AT)1
 U 1 1 5E351885
 P 5550 4500
@@
 	5250 4100 5500 4100
 $Comp
-L BalthazarPSU-rescue:INDUCTOR_SMALL FBEAD3
+L BalthazarPSU-rescue:INDUCTOR_SMALL-BalthazarPSU-rescue FBEAD3
 U 1 1 5EF3D9A1
 P 5950 4100
@@
 	7450 3650 7500 3650
 $Comp
-L BalthazarPSU-rescue:INDUCTOR_SMALL L2
+L BalthazarPSU-rescue:INDUCTOR_SMALL-BalthazarPSU-rescue L2
 U 1 1 5EFF8ED2
 P 7900 1950
@@
 $EndComp
 $Comp
-L BalthazarPSU-rescue:INDUCTOR_SMALL L3
+L BalthazarPSU-rescue:INDUCTOR_SMALL-BalthazarPSU-rescue L3
 U 1 1 5EFF9E33
 P 7900 3200
@@
 	7200 2950 7300 2950
 $Comp
-L BalthazarPSU-rescue:INDUCTOR_SMALL FBEAD2
+L BalthazarPSU-rescue:INDUCTOR_SMALL-BalthazarPSU-rescue FBEAD2
 U 1 1 5EE8BD2A
 P 2050 3250
@@
 $EndComp
 $Comp
-L BalthazarPSU-rescue:BQ24193 IC1
+L BalthazarPSU-rescue:BQ24193-BalthazarPSU-rescue IC1
 U 1 1 5EC6F97C
 P 4650 3950
@@
 Connection ~ 3050 4550
 $Comp
-L Connector:Conn_01x02_Female THERM
+L Connector:Conn_01x02_Female THERM1
 U 1 1 5E94198E
 P 6450 4550
-F 0 "THERM" H 6478 4526 50  0000 L CNN
+F 0 "THERM1" H 6478 4526 50  0000 L CNN
 F 1 "thermistor" H 6478 4435 50  0000 L CNN
 F 2 "TestPoint:TestPoint_2Pads_Pitch2.54mm_Drill0.8mm" H 6450 4550 50  0001 C CNN
@@
 $EndComp
 $Comp
-L BalthazarPSU-rescue:Led_Small D5
+L BalthazarPSU-rescue:Led_Small-BalthazarPSU-rescue D5
 U 1 1 5E93AE8A
 P 7050 3950
@@
 $EndComp
 $Comp
-L BalthazarPSU-rescue:Led_Small D4
+L BalthazarPSU-rescue:Led_Small-BalthazarPSU-rescue D4
 U 1 1 5E9E9310
 P 7050 2700
@@
 	6200 4100 6250 4100
 $Comp
-L Connector:Conn_01x02_Female BATT
+L Connector:Conn_01x02_Female BATT1
 U 1 1 5E8DE18A
 P 6450 4100
-F 0 "BATT" H 6478 4076 50  0000 L CNN
+F 0 "BATT1" H 6478 4076 50  0000 L CNN
 F 1 "1s LiPo" H 6478 3985 50  0000 L CNN
 F 2 "TerminalBlock:TerminalBlock_bornier-2_P5.08mm" H 6450 4100 50  0001 C CNN
